Commit message: HMS_Perception makeover

File: HMS_Perception/src/description/HMS_Perception_description.urdf (robot description, URDF)
Before this commit: robot HMS_Perception, 3 links, 2 joints
Links:
- removed link arm_base_link
- removed link base_footprint
- added link body; collision box size=${body_length} ${body_width} ${body_height}; visual box size=${body_length} ${body_width} ${body_height}
- added link imu_link, mass 0.001; collision box size=.001 .001 .001; visual box size=0.001 0.001 0.001
- link base_link: geometry visual box size=0.05 0.05 0.01
Joints:
- removed joint arm_base_joint
- removed joint base_joint
- added joint base_link_to_chasis: type fixed, parent base_link, child body
- added joint imu_joint: type fixed, parent base_link, child imu_link, origin xyz=0 0 0.05, axis 1 0 0
